Commit message: update the urdf for moma

File: urdf/ur_macro_husky.xacro (robot description, xacro)
@@ -311,5 +311,5 @@
     <joint name="${tf_prefix}base_joint" type="fixed">
       <xacro:insert_block name="origin" />
-      <parent link="${parent}" />
+      <parent link="top_plate_default_mount" />
       <child link="${tf_prefix}base_link" />
     </joint>
